Commit message: 更新了urdf让他可以跑了

File: urdf/car.urdf (robot description, URDF)
Before this commit: robot differential_wheeled_robot, 7 links, 6 joints
Links:
- removed link camera_link
- added link camera_front_link; visual box size=0.02 0.02 0.02
- added link camera_left_link; visual box size=0.02 0.02 0.02
- added link camera_right_link; visual box size=0.02 0.02 0.02
Joints:
- removed joint camera_joint
- added joint camera_front_joint: type fixed, parent hokuyo_link, child camera_front_link, origin xyz=0 0 0.08 rpy=0 0 0
- added joint camera_left_joint: type fixed, parent base_link, child camera_left_link, origin xyz=0.08 0.08 0.08 rpy=0 0 0
- added joint camera_right_joint: type fixed, parent base_link, child camera_right_link, origin xyz=-0.08 0.08 0.08 rpy=0 0 0
- joint hokuyo_joint: origin xyz=0 0 0.1 rpy=0 0 0 -> xyz=0.125 0 0.0325 rpy=0 0 0; parent camera_link -> base_link

Commit message: 完成三个深度摄像头在rviz下的位置问题

File: urdf/car.urdf (robot description, URDF)
Before this commit: robot differential_wheeled_robot, 9 links, 8 joints
Joints:
- joint camera_left_joint: origin xyz=0.08 0.08 0.08 rpy=0 0 0 -> xyz=0.08 0.08 0.08 rpy=0 0 1.57
- joint camera_right_joint: origin xyz=-0.08 0.08 0.08 rpy=0 0 0 -> xyz=0.08 -0.08 0.08 rpy=0 0 -1.57

Commit message: 与linux系统同步

File: urdf/car.urdf (robot description, URDF)
Before this commit: robot differential_wheeled_robot, 9 links, 8 joints
Links:
- link hokuyo_link: geometry collision box size=.05 .05 .05; visual mesh filename=package://autonomus_transport_industrial_system/urdf/meshes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
