Commit message: 调试底盘，可以正常操控了(car.urdf)

File: urdf/car_.urdf (robot description, URDF)
Before this commit: robot differential_wheeled_robot, 9 links, 8 joints
Links:
- removed link camera_front_link
- removed link camera_left_link
- removed link camera_right_link
- removed link caster_back_link
- removed link caster_front_link
- added link back_left_wheel, mass 2.5; collision cylinder length=0.03 radius=0.032; visual cylinder length=0.03 radius=0.032
- added link back_right_wheel, mass 2.5; collision cylinder length=0.03 radius=0.032; visual cylinder length=0.03 radius=0.032
- added link camera_link; visual box size=0.05 0.05 0.05
- added link imu_link_; visual box size=0.05 0.05 0.05
- link base_link: geometry collision box size=0.28 0.17 0.05; visual box size=0.2 0.2 0.05
- link front_left_wheel: geometry collision cylinder length=0.03 radius=0.032; visual cylinder length=0.03 radius=0.032
- link front_right_wheel: geometry collision cylinder length=0.03 radius=0.032; visual cylinder length=0.03 radius=0.032
- link hokuyo_link: geometry collision box size=.05 .05 .05; visual mesh filename=package://gx2019_omni_simulations/urdf/meshes/hokuyo.dae
Joints:
- removed joint camera_front_joint
- removed joint camera_left_joint
- removed joint camera_right_joint
- removed joint caster_back_joint
- removed joint caster_front_joint
- added joint back_left_wheel_joint: type continuous, parent base_link, child back_left_wheel, origin xyz=-0.07 0.095 0.0 rpy=0 0 0, axis 0 1 0, limit effort=100 velocity=100
- added joint back_right_wheel_joint: type continuous, parent base_link, child back_right_wheel, origin xyz=-0.07 -0.095 0.0 rpy=0 0 0, axis 0 1 0, limit effort=100 velocity=100
- added joint camera_joint: type fixed, parent base_link, child camera_link, origin xyz=0 0 0.1 rpy=0 0 -1.57
- added joint imu_joint: type fixed, parent base_link, child imu_link_, origin xyz=0 0 0.05 rpy=0 0 0
- joint front_left_wheel_joint: origin xyz=0.0 0.15 0.0 rpy=0 0 0 -> xyz=0.07 0.095 0.0 rpy=0 0 0
- joint front_right_wheel_joint: origin xyz=0.0 -0.15 0.0 rpy=0 0 0 -> xyz=0.07 -0.095 0.0 rpy=0 0 0
- joint hokuyo_joint: origin xyz=0.125 0 0.0325 rpy=0 0 0 -> xyz=0.065 0 0.0325 rpy=0 0 -3.14

File: urdf/car_apriltag.urdf (robot description, URDF)
Before this commit: robot differential_wheeled_robot, 9 links, 8 joints
Links:
- removed link camera_front_link
- removed link camera_left_link
- removed link camera_right_link
- removed link hokuyo_link
- added link camera_link; visual box size=0.05 0.05 0.05
- link base_link: geometry collision cylinder length=0.02 radius=0.15; visual cylinder length=0.02 radius=0.15
- link caster_back_link: mass 0.0 -> 0.5; geometry collision sphere radius=0.025; visual sphere radius=0.025
- link caster_front_link: mass 0.0 -> 0.5; geometry collision sphere radius=0.025; visual sphere radius=0.025
- link front_left_wheel: geometry collision cylinder length=0.02 radius=0.04; visual cylinder length=0.02 radius=0.04
- link front_right_wheel: geometry collision cylinder length=0.02 radius=0.04; visual cylinder length=0.02 radius=0.04
Joints:
- removed joint camera_front_joint
- removed joint camera_left_joint
- removed joint camera_right_joint
- removed joint hokuyo_joint
- added joint camera_joint: type fixed, parent base_link, child camera_link, origin xyz=0.125 0 0.0325 rpy=0 0 0
- joint caster_back_joint: origin xyz=-0.24 0 -0.05 rpy=-1.57079632679 0 0 -> xyz=-0.135 0.0 0.009 rpy=-1.57079632679 0 0
- joint caster_front_joint: origin xyz=0.24 0 -0.05 rpy=-1.57079632679 0 0 -> xyz=0.115 0.0 0.007 rpy=-1.57079632679 0 0
- joint front_left_wheel_joint: origin xyz=0.0 0.15 0.0 rpy=0 0 0 -> xyz=0.0 -0.15 0.0 rpy=0 0 0
- joint front_right_wheel_joint: origin xyz=0.0 -0.15 0.0 rpy=0 0 0 -> xyz=0.0 0.15 0.0 rpy=0 0 0

Commit message: 添加params文件夹，使用car_.urdf

File: urdf/car_.urdf (robot description, URDF)
Before this commit: robot differential_wheeled_robot, 8 links, 7 joints
Links:
- removed link camera_link
- added link camera_front_link; visual box size=0.02 0.02 0.02
- added link camera_left_link; visual box size=0.02 0.02 0.02
- added link camera_right_link; visual box size=0.02 0.02 0.02
Joints:
- removed joint camera_joint
- added joint camera_front_joint: type fixed, parent hokuyo_link, child camera_front_link, origin xyz=0 0 0.08 rpy=0 0 0
- added joint camera_left_joint: type fixed, parent base_link, child camera_left_link, origin xyz=0.08 0.08 0.08 rpy=0 0 1.57
- added joint camera_right_joint: type fixed, parent base_link, child camera_right_link, origin xyz=0.08 -0.08 0.08 rpy=0 0 -1.57

Commit message: 使用新型小车

File: urdf/car_.urdf (robot description, URDF)
Before this commit: robot differential_wheeled_robot, 10 links, 9 joints
Links:
- link hokuyo_link: geometry collision box size=.05 .05 .05; visual mesh filename=package://autonomus_transport_industrial_system/urdf/meshes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

File: urdf/robot1.urdf (robot description, URDF)
Before this commit: robot robot, 27 links, 26 joints
Links:
- added link camera_front_link; visual mesh filename=package://autonomus_transport_industrial_system/urdf/meshes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
- added link hokuyo_link, mass 1e-5; collision box size=.05 .05 .05; visual mesh filename=package://autonomus_transport_industrial_system/urdf/meshes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
- link back_wheel: mass None -> 2.5; geometry collision sphere radius=0.03; visual sphere radius=0.03
- link forward_wheel: mass None -> 2.5; geometry collision sphere radius=0.03; visual sphere radius=0.03
- link forward_wheel_base: mass None -> 2.5; geometry collision cylinder length=0.03 radius=0.032; visual box size=0.05 0.05 0.0325
- link left_wheel: mass None -> 2.5; geometry collision cylinder length=0.03 radius=0.03; visual cylinder length=0.03 radius=0.03
- link right_wheel: mass None -> 2.5; geometry collision cylinder length=0.03 radius=0.03; visual cylinder length=0.03 radius=0.03
Joints:
- added joint camera_front_joint: type fixed, parent base_link, child camera_front_link, origin xyz=0.06 0.0 0.10 rpy=0.0 0.15 0
- added joint hokuyo_joint: type fixed, parent base_link, child hokuyo_link, origin xyz=0.06 0 0.03 rpy=0 0 -3.14, axis 0 1 0
- joint left_motor_to_left_wheel: origin xyz=0 0.045 0 rpy=0 0 0 -> xyz=0 0.1 -0.035 rpy=0 0 0; parent left_motor -> base_link
- joint right_motor_to_right_wheel: origin xyz=0 -0.045 0 rpy=0 0 0 -> xyz=0 -0.1 -0.035 rpy=0 0 0; parent right_motor -> base_link
