Commit message: 能够使用rtabmap完成建图，导航

File: urdf/robot1.urdf (robot description, URDF)
Before this commit: robot robot, 29 links, 28 joints
Links:
- added link imu_link; visual box size=0.05 0.05 0.0325
Joints:
- added joint imu_joint: type fixed, parent base_link, child imu_link, origin xyz=0.0 0.0 0.1 rpy=0.0 0 0

Commit message: 启用rgbd_odometry

File: urdf/robot1.urdf (robot description, URDF)
Before this commit: robot robot, 30 links, 29 joints
Links:
- link back_wheel: mass 2.5 -> None
- link forward_wheel_base: mass 2.5 -> None
Joints:
- joint camera_front_joint: origin xyz=0.06 0.0 0.10 rpy=0.0 0.15 0 -> xyz=0.06 0.0 0.05 rpy=0.0 0.15 0
