Commit message: 使用简洁模型robot.urdf，tf树正确

File: urdf/robot.urdf (robot description, URDF)
Before this commit: robot robot, 15 links, 14 joints
Links:
- removed link back_wheel
- removed link back_wheel_base
- removed link left_fix
- removed link left_fix2
- removed link left_fix3
- removed link left_fix4
- removed link left_motor
- removed link left_wheel
- removed link right_fix
- removed link right_fix2
- removed link right_fix3
- removed link right_fix4
- removed link right_motor
- removed link right_wheel
- added link camera_front_link; visual mesh filename=package://autonomus_transport_industrial_system/urdf/meshes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
- added link caster_back_link, mass 0.5; collision sphere radius=0.028; visual sphere radius=0.028
- added link caster_front_link, mass 0.5; collision sphere radius=0.026; visual sphere radius=0.026
- added link front_left_wheel, mass 2.5; collision cylinder length=0.02 radius=0.04; visual cylinder length=0.02 radius=0.04
- added link front_right_wheel, mass 2.5; collision cylinder length=0.02 radius=0.04; visual cylinder length=0.02 radius=0.04
- added link hokuyo_link, mass 1e-5; collision box size=.05 .05 .05; visual mesh filename=package://autonomus_transport_industrial_system/urdf/meshes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
- link base_link: mass None -> 5; geometry collision cylinder length=0.02 radius=0.15; visual cylinder length=0.02 radius=0.15
Joints:
- removed joint back_wheel_to_back_wheel_base
- removed joint back_wheel_to_base_link
- removed joint base_link_to_left_motor
- removed joint base_link_to_right_motor
- removed joint left_fix2_to_left_fix
- removed joint left_fix3_to_base_link
- removed joint left_fix4_to_left_fix3
- removed joint left_fix_to_base_link
- removed joint left_motor_to_left_wheel
- removed joint right_fix2_to_right_fix
- removed joint right_fix3_to_base_link
- removed joint right_fix4_to_right_fix3
- removed joint right_fix_to_base_link
- removed joint right_motor_to_right_wheel
- added joint camera_front_joint: type fixed, parent base_link, child camera_front_link, origin xyz=0.06 0.0 0.15 rpy=0.0 0.15 0
- added joint caster_back_joint: type fixed, parent base_link, child caster_back_link, origin xyz=-0.135 0.0 0.008 rpy=-1.57079632679 0 0
- added joint caster_front_joint: type fixed, parent base_link, child caster_front_link, origin xyz=0.115 0.0 0.008 rpy=-1.57079632679 0 0
- added joint front_left_wheel_joint: type continuous, parent base_link, child front_left_wheel, origin xyz=0.0 -0.15 0.0 rpy=0 0 0, axis 0 1 0, limit effort=100 velocity=100
- added joint front_right_wheel_joint: type continuous, parent base_link, child front_right_wheel, origin xyz=0.0 0.15 0.0 rpy=0 0 0, axis 0 1 0, limit effort=100 velocity=100
- added joint hokuyo_joint: type fixed, parent base_link, child hokuyo_link, origin xyz=0.06 0 0.08 rpy=0 0 -3.14, axis 0 1 0

File: urdf/robot1.urdf (robot description, URDF)
Before this commit: robot robot, 30 links, 29 joints
Joints:
- removed joint left_motor_to_left_wheel
- removed joint right_motor_to_right_wheel
- added joint base_link_to_left_wheel: type continuous, parent base_link, child left_wheel, origin xyz=0 0.1 -0.035 rpy=0 0 0, axis 0 1 0
- added joint base_link_to_right_wheel: type continuous, parent base_link, child right_wheel, origin xyz=0 -0.1 -0.035 rpy=0 0 0, axis 0 1 0
